Commit message: fix base_link

File: irobot_create_description/urdf/create3.urdf.xacro (robot description, xacro)
@@ -11,18 +11,18 @@
   <xacro:include filename="$(find irobot_create_description)/urdf/wheel_with_wheeldrop.urdf.xacro" />
   <!-- MECHANICAL PROPERTIES -->
-  <xacro:property name="body_z_offset"           value="${4.1*cm2m}" />
-  <xacro:property name="body_collision_z_offset" value="${1*cm2m}" />
+  <xacro:property name="body_z_offset"           value="${-2.5*cm2m}" />
+  <xacro:property name="body_collision_z_offset" value="${-1*cm2m}" />
   <xacro:property name="body_mass"               value="2.300" />
   <xacro:property name="body_radius"             value="${16.4*cm2m}" />
   <xacro:property name="body_length"             value="${6*cm2m}" />
   <xacro:property name="bumper_mass"             value="0.1" />
-  <xacro:property name="bumper_offset_z"         value="${4.1*cm2m}" />
+  <xacro:property name="bumper_offset_z"         value="${-2.5*cm2m}" />
   <xacro:property name="bumber_inertial_x"       value="${8*cm2m}" />
   <xacro:property name="bumper_inertial_z"       value="${2*cm2m}"/>
-  <xacro:property name="wheel_height"            value="${3.85*cm2m}" />
+  <xacro:property name="wheel_height"            value="${-2.75*cm2m}" />
   <xacro:property name="distance_between_wheels" value="${23.3*cm2m}" />
   <xacro:property name="caster_position_x"       value="${12.5*cm2m}" />
-  <xacro:property name="caster_position_z"       value="${1.2*cm2m}" />
-  <xacro:property name="wheel_drop_offset_z"     value="${3.1*mm2m}"/>
+  <xacro:property name="caster_position_z"       value="${-5.4*cm2m}" />
+  <xacro:property name="wheel_drop_offset_z"     value="${3.5*mm2m}"/>
   <xacro:property name="wheel_drop_z"            value="${wheel_height + wheel_drop_offset_z}"/>
   <!-- Create 3 base definition-->

Commit message: Fixed robot collision z offset; Prevent slipping

File: irobot_create_description/urdf/create3.urdf.xacro (robot description, xacro)
@@ -12,5 +12,5 @@
   <!-- MECHANICAL PROPERTIES -->
   <xacro:property name="body_z_offset"           value="${-2.5*cm2m}" />
-  <xacro:property name="body_collision_z_offset" value="${-1*cm2m}" />
+  <xacro:property name="body_collision_z_offset" value="${1*cm2m}" />
   <xacro:property name="body_mass"               value="2.300" />
   <xacro:property name="body_radius"             value="${16.4*cm2m}" />

Commit message: Fixed caster height

File: irobot_create_description/urdf/create3.urdf.xacro (robot description, xacro)
@@ -23,8 +23,9 @@
   <xacro:property name="distance_between_wheels" value="${23.3*cm2m}" />
   <xacro:property name="caster_position_x"       value="${12.5*cm2m}" />
-  <xacro:property name="caster_position_z"       value="${-5.4*cm2m}" />
+  <xacro:property name="caster_position_z"       value="${-5.55*cm2m}" />
   <xacro:property name="wheel_drop_offset_z"     value="${3.5*mm2m}"/>
   <xacro:property name="wheel_drop_z"            value="${wheel_height + wheel_drop_offset_z}"/>
   <!-- Create 3 base definition-->
+  <origin xyz="0 0 0.064171"/>
   <link name="base_link">
     <visual>
